File: hardware/BioAmp-EXG-Pill.kicad_sch (KiCad schematic)
At the start: 27 parts, among them J1 BioAmp Output, J2 BioAmp Input, U1 Amp, U2 LOGO_UDLABS

Commit message: commint inicial
borrar logo
Parts:
- removed U2: LOGO_UDLABS, udlabs:EXG, symbol BioAmp-EXG-Pill-rescue:LOGO_UDLABS-udlabs
- C1: renamed from C4; value 1nF -> 2.2nF
- C2: renamed from R4; value 220K -> 47nF; footprint Resistor_SMD:R_0603_1608Metric_Pad0.98x0.95mm_HandSolder -> Capacitor_SMD:C_0603_1608Metric_Pad1.08x0.95mm_HandSolder; symbol Device:R -> Device:C
- C3: renamed from C2; value 1nF -> 47nF
- C5: renamed from C7; value 10uF -> 4.7uF
- C7: renamed from C3; value 10uF -> 220nF
- R13: renamed from R8; value 1M -> 10K
- R14: renamed from R11; value 0R -> 1k
- R15: renamed from R9; value 1M -> 10K
- R4: renamed from R5; value 22K -> 1K
- R5: renamed from R10; value 220K -> 10K
- R8: renamed from R2; value 220K -> 10K
- R9: renamed from R7; value 22K -> 1K
- U1: value Amp -> TL074
- renumbered C6 to C4, C1 to C6, C5 to C8, JP2 to JP1, JP1 to JP2, R6 to R1, R3 to R11, R1 to R12, R13 to R2, R12 to R3, R14 to R6
Connections:
- net bpfOUT renamed OUT
Other:
- note added: "1000x Gain (Bandpass)"
- note added: "Bridge all three pads of the solder jumper to configure for 2 Electrode operations instead of the 3 electrodes Note: 2 electrodes will give noisier output than 3 electrodes!"
- note added: "C8 (BPFC_C) & R3 (BPFC_R) on the back side of the PCB can be used to configure the bandpass filter. Use them to configure output Gain (decrease) & Band (frequency range)."
- note added: "Create solder joint on JP2 to narrow the Band Pass freqnecny range Default: Wide input frequency band, use when recording EMG, EOG Configured: Narrow input frequency band, use for EEG, EOG, and ECG"
- note added: "Instrumentation Amp (INA)"
- note added: "Narrow Band"
- note removed: "1000x Gain Bandpass Filter"
- note removed: "11x Gain Instrumentation Amp (INA)"
- note removed: "Bridge all three pads of the solder jumper (JP2) to configure for 2 Electrode operations instead of the 3 electrodes Note: 2 electrodes will give noisier output than 3 electrodes!"
- note removed: "C5 (BPFC_C) & R12 (BPFC_R) on the back side of the PCB can be used to configure the bandpass filter. Use them to configure output Gain (decrease) & Band (frequency range)."
- note removed: "Create solder joint on JP1 to increase the Band Pass freqnecny range Default: Narrow input frequency band, use when recording EEG, EOG Configured: Wide input frequency band, use for ECG, EMG, and EOG"
- note removed: "Wide Band"
- moved on the sheet: J1, R5
